File: Pteron56v0/Pteron56v0.kicad_pcb (KiCad board)
At the start: 2 copper layers, 293.7 x 154 mm, 135 parts, among them SW1 SW_PUSH, SW10 SW_PUSH, SW11 SW_PUSH, SW12 SW_PUSH, SW13 SW_PUSH, SW14 SW_PUSH, SW15 SW_PUSH, SW16 SW_PUSH, SW17 SW_PUSH, SW18 SW_PUSH, SW19 SW_PUSH, SW2 SW_PUSH, SW20 SW_PUSH, SW21 SW_PUSH, SW22 SW_PUSH, SW23 SW_PUSH, SW24 SW_PUSH, SW25 SW_PUSH, SW26 SW_PUSH, SW27 SW_PUSH, SW28 SW_PUSH, SW29 SW_PUSH, SW3 SW_PUSH, SW30 SW_PUSH, SW31 SW_PUSH, SW32 SW_PUSH, SW33 SW_PUSH, SW34 SW_PUSH, SW35 SW_PUSH, SW36 SW_PUSH, SW37 SW_PUSH, SW38 SW_PUSH, SW39 SW_PUSH, SW4 SW_PUSH, SW40 SW_PUSH, SW41 SW_PUSH, SW42 SW_PUSH, SW43 SW_PUSH, SW44 SW_PUSH, SW45 SW_PUSH, SW46 SW_PUSH, SW47 SW_PUSH, SW48 SW_PUSH, SW49 SW_PUSH, SW5 SW_PUSH, SW50 SW_PUSH, SW51 SW_PUSH, SW52 SW_PUSH, SW53 SW_PUSH, SW54 SW_PUSH, SW55 SW_PUSH, SW56 SW_PUSH, SW6 SW_PUSH, SW7 SW_PUSH, SW8 SW_PUSH, SW9 SW_PUSH, U1 ProMicro

Commit message: Add files via upload
More edits, finished the MCU. 

TODO:
THT LEDs
WS2812b underglow
Add EC11 encoder
Parts:
- removed the REF** at (259.7, 71.4)
- removed the REF** at (68.6, 134.8)
- removed the REF** at (128.5, 176.1)
- removed the REF** at (162.4, 176.2)
- removed the REF** at (222.3, 134.8)
- removed the REF** at (289.1, 103.9)
- removed the REF** at (268.9, 28.6)
- removed the REF** at (200.0, 32.7)
- removed the REF** at (90.9, 32.7)
- removed the REF** at (220.0, 70.3)
- removed the REF** at (184.4, 84.7)
- removed the REF** at (176.1, 130.4)
- removed the REF** at (114.8, 130.4)
- removed the REF** at (106.5, 84.8)
- removed the REF** at (71.0, 70.2)
- removed the REF** at (31.2, 71.5)
- removed the REF** at (1.80, 104.0)
- added C1: 22p, Keyboard parts:22pf_0603, F.Cu at (175.4, 80.2)
- added C2: .1u, Keyboard parts:.1uf_0805, F.Cu at (193.0, 66.0)
- added C3: .1u, Keyboard parts:.1uf_0805, F.Cu at (187.4, 78.1)
- added C4: 22p, Keyboard parts:22pf_0603, F.Cu at (172.7, 77.0)
- added C5: .1u, Keyboard parts:.1uf_0805, F.Cu at (172.5, 71.8)
- added C6: 1u, Keyboard parts:.1uf_0805, F.Cu at (178.5, 62.1)
- added C7: 10u, Keyboard parts:.1uf_0805, F.Cu at (187.5, 59.3)
- added D100: LED, LED_SMD:LED_0402_1005Metric, F.Cu at (196.2, 12.2)
- added D101: LED, LED_SMD:LED_0402_1005Metric, F.Cu at (213.5, -3.83)
- added D102: LED, LED_SMD:LED_0402_1005Metric, F.Cu at (201.0, 8.14)
- added D103: LED, LED_SMD:LED_0402_1005Metric, F.Cu at (207.6, 1.17)
- added D104: LED, LED_SMD:LED_0402_1005Metric, F.Cu at (192.2, 15.4)
- added D105: LED, LED_SMD:LED_0402_1005Metric, F.Cu at (203.1, 5.13)
- added D106: LED, LED_SMD:LED_0402_1005Metric, F.Cu at (207.6, -0.82)
- added D107: LED, LED_SMD:LED_0402_1005Metric, F.Cu at (210.7, 0.15)
- added D108: LED, LED_SMD:LED_0402_1005Metric, F.Cu at (202.5, 12.1)
- added D109: LED, LED_SMD:LED_0402_1005Metric, F.Cu at (207.3, 7.14)
- added D110: LED, LED_SMD:LED_0402_1005Metric, F.Cu at (209.4, 5.15)
- added D111: LED, LED_SMD:LED_0402_1005Metric, F.Cu at (199.3, 14.2)
- added D112: LED, LED_SMD:LED_0402_1005Metric, F.Cu at (213.8, 0.15)
- added D57: LED, LED_SMD:LED_0402_1005Metric, F.Cu at (196.8, 4.16)
- added D58: LED, LED_SMD:LED_0402_1005Metric, F.Cu at (207.2, -6.79)
- added D59: LED, LED_SMD:LED_0402_1005Metric, F.Cu at (189.9, 12.5)
- added D60: LED, LED_SMD:LED_0402_1005Metric, F.Cu at (201.3, 1.15)
- added D61: LED, LED_SMD:LED_0402_1005Metric, F.Cu at (207.2, -4.80)
- added D62: LED, LED_SMD:LED_0402_1005Metric, F.Cu at (191.6, 9.46)
- added D63: LED, LED_SMD:LED_0402_1005Metric, F.Cu at (213.8, -1.84)
- added D64: LED, LED_SMD:LED_0402_1005Metric, F.Cu at (210.4, 7.14)
- added D65: LED, LED_SMD:LED_0402_1005Metric, F.Cu at (202.5, 14.1)
- added D66: LED, LED_SMD:LED_0402_1005Metric, F.Cu at (212.5, 4.13)
- added D67: LED, LED_SMD:LED_0402_1005Metric, F.Cu at (207.3, 9.13)
- added D68: LED, LED_SMD:LED_0402_1005Metric, F.Cu at (212.5, 2.14)
- added D69: LED, LED_SMD:LED_0402_1005Metric, F.Cu at (211.6, -9.80)
- added D70: LED, LED_SMD:LED_0402_1005Metric, F.Cu at (194.7, 9.22)
- added D71: LED, LED_SMD:LED_0402_1005Metric, F.Cu at (211.6, -7.81)
- added D72: LED, LED_SMD:LED_0402_1005Metric, F.Cu at (200.0, 4.16)
- added D73: LED, LED_SMD:LED_0402_1005Metric, F.Cu at (189.0, 15.0)
- added D74: LED, LED_SMD:LED_0402_1005Metric, F.Cu at (214.8, -9.80)
- added D75: LED, LED_SMD:LED_0402_1005Metric, F.Cu at (207.2, -2.81)
- added D76: LED, LED_SMD:LED_0402_1005Metric, F.Cu at (204.4, 1.15)
- added D77: LED, LED_SMD:LED_0402_1005Metric, F.Cu at (193.0, 11.5)
- added D78: LED, LED_SMD:LED_0402_1005Metric, F.Cu at (185.9, 15.0)
- added D79: LED, LED_SMD:LED_0402_1005Metric, F.Cu at (196.7, 6.21)
- added D80: LED, LED_SMD:LED_0402_1005Metric, F.Cu at (199.8, 6.15)
- added D81: LED, LED_SMD:LED_0402_1005Metric, F.Cu at (197.9, 8.20)
- added D82: LED, LED_SMD:LED_0402_1005Metric, F.Cu at (210.3, -3.83)
- added D83: LED, LED_SMD:LED_0402_1005Metric, F.Cu at (193.0, 13.4)
- added D84: LED, LED_SMD:LED_0402_1005Metric, F.Cu at (214.8, -7.81)
- added D85: LED, LED_SMD:LED_0402_1005Metric, F.Cu at (203.1, 3.14)
- added D86: LED, LED_SMD:LED_0402_1005Metric, F.Cu at (197.9, 10.2)
- added D87: LED, LED_SMD:LED_0402_1005Metric, F.Cu at (210.3, -5.82)
- added D88: LED, LED_SMD:LED_0402_1005Metric, F.Cu at (204.1, 9.13)
- added D89: LED, LED_SMD:LED_0402_1005Metric, F.Cu at (195.3, 16.2)
- added D90: LED, LED_SMD:LED_0402_1005Metric, F.Cu at (209.4, 3.16)
- added D91: LED, LED_SMD:LED_0402_1005Metric, F.Cu at (213.5, -5.82)
- added D92: LED, LED_SMD:LED_0402_1005Metric, F.Cu at (204.1, 7.14)
- added D93: LED, LED_SMD:LED_0402_1005Metric, F.Cu at (199.3, 12.2)
- added D94: LED, LED_SMD:LED_0402_1005Metric, F.Cu at (206.3, 5.15)
- added D95: LED, LED_SMD:LED_0402_1005Metric, F.Cu at (206.3, 3.16)
- added D96: LED, LED_SMD:LED_0402_1005Metric, F.Cu at (196.2, 14.2)
- added D97: LED, LED_SMD:LED_0402_1005Metric, F.Cu at (198.5, 16.2)
- added D98: LED, LED_SMD:LED_0402_1005Metric, F.Cu at (201.0, 10.1)
- added D99: LED, LED_SMD:LED_0402_1005Metric, F.Cu at (210.7, -1.84)
- added F1: 500mA, Fuse:Fuse_0402_1005Metric, F.Cu at (186.5, 50.8)
- added J1: USB_C_Receptacle_USB2.0, Connector_USB:USB_C_Receptacle_XKB_U262-16XN-4BVC11, F.Cu at (183.2, 45.3)
- added Q1: 2N2219, Package_TO_SOT_THT:TO-39-3, F.Cu at (197.5, -5.32)
- added R1: 5.1k, Resistor_SMD:R_0603_1608Metric, F.Cu at (186.4, 52.8)
- added R10: 1k, Resistor_SMD:R_0805_2012Metric, F.Cu at (255.5, -13.4)
- added R11: 1k, Resistor_SMD:R_0805_2012Metric, F.Cu at (260.0, -16.4)
- added R12: 1k, Resistor_SMD:R_0805_2012Metric, F.Cu at (251.1, -7.51)
- added R13: 1k, Resistor_SMD:R_0805_2012Metric, F.Cu at (255.5, -10.5)
- added R14: 1k, Resistor_SMD:R_0805_2012Metric, F.Cu at (260.0, -13.4)
- added R15: 1k, Resistor_SMD:R_0805_2012Metric, F.Cu at (264.4, -16.4)
- added R16: 1k, Resistor_SMD:R_0805_2012Metric, F.Cu at (251.1, -4.56)
- added R17: 1k, Resistor_SMD:R_0805_2012Metric, F.Cu at (255.5, -7.51)
- added R18: 1k, Resistor_SMD:R_0805_2012Metric, F.Cu at (260.0, -10.5)
- added R19: 1k, Resistor_SMD:R_0805_2012Metric, F.Cu at (264.4, -13.4)
- added R2: 5.1k, Resistor_SMD:R_0603_1608Metric, F.Cu at (179.7, 52.7)
- added R20: 1k, Resistor_SMD:R_0805_2012Metric, F.Cu at (251.1, -1.61)
- added R21: 1k, Resistor_SMD:R_0805_2012Metric, F.Cu at (251.1, -13.4)
- added R22: 1k, Resistor_SMD:R_0805_2012Metric, F.Cu at (255.5, -4.56)
- added R23: 1k, Resistor_SMD:R_0805_2012Metric, F.Cu at (260.0, -7.51)
- added R24: 1k, Resistor_SMD:R_0805_2012Metric, F.Cu at (264.4, -10.5)
- added R25: 1k, Resistor_SMD:R_0805_2012Metric, F.Cu at (251.1, 1.34)
- added R26: 1k, Resistor_SMD:R_0805_2012Metric, F.Cu at (268.8, -13.4)
- added R27: 1k, Resistor_SMD:R_0805_2012Metric, F.Cu at (255.5, -1.61)
- added R28: 1k, Resistor_SMD:R_0805_2012Metric, F.Cu at (273.2, -16.4)
- added R29: 1k, Resistor_SMD:R_0805_2012Metric, F.Cu at (260.0, -4.56)
- added R3: 10k, Keyboard parts:R_0805, F.Cu at (189.2, 82.1)
- added R30: 1k, Resistor_SMD:R_0805_2012Metric, F.Cu at (264.4, -7.51)
- added R31: 1k, Resistor_SMD:R_0805_2012Metric, F.Cu at (268.8, -10.5)
- added R32: 1k, Resistor_SMD:R_0805_2012Metric, F.Cu at (255.5, 1.34)
- added R33: 1k, Resistor_SMD:R_0805_2012Metric, F.Cu at (273.2, -13.4)
- added R34: 1k, Resistor_SMD:R_0805_2012Metric, F.Cu at (260.0, -1.61)
- added R35: 1k, Resistor_SMD:R_0805_2012Metric, F.Cu at (273.2, -4.56)
- added R36: 1k, Resistor_SMD:R_0805_2012Metric, F.Cu at (264.4, -4.56)
- added R37: 1k, Resistor_SMD:R_0805_2012Metric, F.Cu at (268.8, -7.51)
- added R38: 1k, Resistor_SMD:R_0805_2012Metric, F.Cu at (273.2, -10.5)
- added R39: 1k, Resistor_SMD:R_0805_2012Metric, F.Cu at (260.0, 1.34)
- added R4: 22, Keyboard parts:R_0805, F.Cu at (181.7, 57.0)
- added R40: 1k, Resistor_SMD:R_0805_2012Metric, F.Cu at (277.6, -13.4)
- added R41: 1k, Resistor_SMD:R_0805_2012Metric, F.Cu at (264.4, -1.61)
- added R42: 1k, Resistor_SMD:R_0805_2012Metric, F.Cu at (282.0, -16.4)
- added R43: 1k, Resistor_SMD:R_0805_2012Metric, F.Cu at (268.8, -4.56)
- added R44: 1k, Resistor_SMD:R_0805_2012Metric, F.Cu at (273.2, -7.51)
- added R45: 1k, Resistor_SMD:R_0805_2012Metric, F.Cu at (277.6, -10.5)
- added R46: 1k, Resistor_SMD:R_0805_2012Metric, F.Cu at (264.4, 1.34)
- added R47: 1k, Resistor_SMD:R_0805_2012Metric, F.Cu at (282.0, -13.4)
- added R48: 1k, Resistor_SMD:R_0805_2012Metric, F.Cu at (268.8, -1.61)
- added R49: 1k, Resistor_SMD:R_0805_2012Metric, F.Cu at (277.6, -16.4)
- added R5: 22, Keyboard parts:R_0805, F.Cu at (184.7, 57.0)
- added R50: 1k, Resistor_SMD:R_0805_2012Metric, F.Cu at (286.4, -16.4)
- added R51: 1k, Resistor_SMD:R_0805_2012Metric, F.Cu at (277.6, -7.51)
- added R52: 1k, Resistor_SMD:R_0805_2012Metric, F.Cu at (282.0, -10.5)
- added R53: 1k, Resistor_SMD:R_0805_2012Metric, F.Cu at (268.8, 1.34)
- added R54: 1k, Resistor_SMD:R_0805_2012Metric, F.Cu at (286.4, -13.4)
- added R55: 1k, Resistor_SMD:R_0805_2012Metric, F.Cu at (273.2, -1.61)
- added R56: 1k, Resistor_SMD:R_0805_2012Metric, F.Cu at (277.6, -4.56)
- added R57: 1k, Resistor_SMD:R_0805_2012Metric, F.Cu at (282.0, -7.51)
- added R58: 1k, Resistor_SMD:R_0805_2012Metric, F.Cu at (286.4, -10.5)
- added R59: 1k, Resistor_SMD:R_0805_2012Metric, F.Cu at (273.2, 1.34)
- added R6: 10k, Keyboard parts:R_0805, F.Cu at (194.2, 69.3)
- added R60: 1k, Resistor_SMD:R_0805_2012Metric, F.Cu at (277.6, -1.61)
- added R61: 1k, Resistor_SMD:R_0805_2012Metric, F.Cu at (282.0, -4.56)
- added R62: 1k, Resistor_SMD:R_0805_2012Metric, F.Cu at (286.4, -7.51)
- added R63: 1k, Resistor_SMD:R_0805_2012Metric, F.Cu at (268.8, -16.4)
- added R7: 10k, Resistor_SMD:R_0805_2012Metric, F.Cu at (251.1, -16.4)
- added R8: 1k, Resistor_SMD:R_0805_2012Metric, F.Cu at (255.5, -16.4)
- added R9: 1k, Resistor_SMD:R_0805_2012Metric, F.Cu at (251.1, -10.5)
- added REF**: MountingHole_2mm, MountingHole:MountingHole_2mm, F.Cu at (222.3, 78.1)
- added REF**: MountingHole_2mm, MountingHole:MountingHole_2mm, F.Cu at (39.8, 97.4)
- added REF**: MountingHole_2mm, MountingHole:MountingHole_2mm, F.Cu at (106.5, 128.2)
- added REF**: MountingHole_2mm, MountingHole:MountingHole_2mm, F.Cu at (260.3, 128.2)
- added REF**: MountingHole_2mm, MountingHole:MountingHole_2mm, F.Cu at (327.0, 97.3)
- added REF**: MountingHole_2mm, MountingHole:MountingHole_2mm, F.Cu at (237.9, 26.0)
- added REF**: MountingHole_2mm, MountingHole:MountingHole_2mm, F.Cu at (200.3, 169.6)
- added REF**: MountingHole_2mm, MountingHole:MountingHole_2mm, F.Cu at (128.8, 26.0)
- added REF**: MountingHole_2mm, MountingHole:MountingHole_2mm, F.Cu at (306.8, 22.0)
- added REF**: MountingHole_2mm, MountingHole:MountingHole_2mm, F.Cu at (108.9, 63.6)
- added REF**: MountingHole_2mm, MountingHole:MountingHole_2mm, F.Cu at (166.4, 169.5)
- added REF**: MountingHole_2mm, MountingHole:MountingHole_2mm, F.Cu at (69.2, 64.9)
- added REF**: MountingHole_2mm, MountingHole:MountingHole_2mm, F.Cu at (297.6, 64.8)
- added REF**: MountingHole_2mm, MountingHole:MountingHole_2mm, F.Cu at (214.1, 123.8)
- added REF**: MountingHole_2mm, MountingHole:MountingHole_2mm, F.Cu at (257.9, 63.7)
- added REF**: MountingHole_2mm, MountingHole:MountingHole_2mm, F.Cu at (152.7, 123.8)
- added REF**: MountingHole_2mm, MountingHole:MountingHole_2mm, F.Cu at (144.5, 78.2)
- added SW57: SW_PUSH, Keyboard parts:SW_SPST_TL3342, F.Cu at (183.5, 83.5)
- added U2: ATmega32U4-AU, Package_QFP:TQFP-44_10x10mm_P0.8mm, F.Cu at (183.6, 69.4)
- added X1: XTAL_GND, Keyboard parts:crystal_FA238-TSX3225, F.Cu at (175.5, 76.9)
- SW1, SW10, SW11, SW12, SW13, SW14, SW15, SW16, SW17, SW18, SW19, SW2, SW20, SW21, SW22, SW23, SW24, SW25, SW26, SW27, SW28, SW29, SW3, SW30, SW31, SW32, SW33, SW34, SW35, SW36, SW37, SW38, SW39, SW4, SW40, SW41, SW42, SW43, SW44, SW45, SW46, SW47, SW48, SW49, SW5, SW50, SW51, SW52, SW53, SW54, SW55, SW56, SW6, SW7, SW8, SW9: footprint Keyboard parts:Mx_Alps_100 -> Keyboard parts:MXOnly-1U
- U1: value ProMicro -> USBLC6-2SC6; footprint Keyboard parts:Pro_Micro -> Package_TO_SOT_SMD:SOT-23-6
- moved U1 75.3 mm to (183.2, 53.2), turned to 90 degrees
- moved G*** 39.9 mm to (183.8, 132.4)
- moved G*** 39.7 mm to (183.7, 132.4)
- moved G*** 39.1 mm to (183.9, 103.9)
- moved G*** 38.9 mm to (183.8, 103.8)
- moved D11 38.5 mm to (252.2, 42.6)
- moved D56 38.5 mm to (103.1, 114.4)
- moved SW15 38.5 mm to (211.5, 139.9)
- moved SW32 38.5 mm to (146.0, 109.2)
- moved SW26 38.5 mm to (210.9, 72.4)
- moved D1 38.5 mm to (291.7, 42.3)
- moved D33 38.5 mm to (152.9, 47.2)
- moved SW30 38.5 mm to (155.9, 72.4)
- moved SW24 38.5 mm to (238.7, 102.4)
- moved D22 38.5 mm to (220.8, 72.3)
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Connections:
- D1 pad 1: /Col0 -> Col0
- D10 pad 1: /Col1 -> Col1
- D11 pad 1: /Col2 -> Col2
- D12 pad 1: /Col2 -> Col2
- D13 pad 1: /Col2 -> Col2
- D14 pad 1: /Col2 -> Col2
- D15 pad 1: /Col2 -> Col2
- D16 pad 1: /Col3 -> Col3
- D17 pad 1: /Col3 -> Col3
- D18 pad 1: /Col3 -> Col3
- D19 pad 1: /Col3 -> Col3
- D2 pad 1: /Col0 -> Col0
- D20 pad 1: /Col3 -> Col3
- D21 pad 1: /Col4 -> Col4
- D22 pad 1: /Col4 -> Col4
- D23 pad 1: /Col4 -> Col4
- D24 pad 1: /Col4 -> Col4
- D25 pad 1: /Col5 -> Col5
- D26 pad 1: /Col5 -> Col5
- D27 pad 1: /Col5 -> Col5
- D28 pad 1: /Col5 -> Col5
- D29 pad 1: /Col6 -> Col6
- D3 pad 1: /Col0 -> Col0
- D30 pad 1: /Col6 -> Col6
- D31 pad 1: /Col6 -> Col6
- D32 pad 1: /Col6 -> Col6
- D33 pad 1: /Col7 -> Col7
- D34 pad 1: /Col7 -> Col7
- D35 pad 1: /Col7 -> Col7
- D36 pad 1: /Col7 -> Col7
- D37 pad 1: /Col8 -> Col8
- D38 pad 1: /Col8 -> Col8
- D39 pad 1: /Col8 -> Col8
- D4 pad 1: /Col0 -> Col0
- D40 pad 1: /Col8 -> Col8
- D41 pad 1: /Col8 -> Col8
- D42 pad 1: /Col9 -> Col9
- D43 pad 1: /Col9 -> Col9
- D44 pad 1: /Col9 -> Col9
- D45 pad 1: /Col9 -> Col9
- D46 pad 1: /Col9 -> Col9
- D47 pad 1: /Col10 -> Col10
- D48 pad 1: /Col10 -> Col10
- D49 pad 1: /Col10 -> Col10
- D5 pad 1: /Col0 -> Col0
- D50 pad 1: /Col10 -> Col10
- D51 pad 1: /Col10 -> Col10
- D52 pad 1: /Col11 -> Col11
- D53 pad 1: /Col11 -> Col11
- D54 pad 1: /Col11 -> Col11
- D55 pad 1: /Col11 -> Col11
- D56 pad 1: /Col11 -> Col11
- D6 pad 1: /Col1 -> Col1
- D7 pad 1: /Col1 -> Col1
- D8 pad 1: /Col1 -> Col1
- D9 pad 1: /Col1 -> Col1
- SW1 pad 1: /Row0 -> Row0
- SW10 pad 1: /Row4 -> Row4
- SW11 pad 1: /Row0 -> Row0
- SW12 pad 1: /Row1 -> Row1
- SW13 pad 1: /Row2 -> Row2
- SW14 pad 1: /Row3 -> Row3
- SW15 pad 1: /Row4 -> Row4
- SW16 pad 1: /Row0 -> Row0
- SW17 pad 1: /Row1 -> Row1
- SW18 pad 1: /Row2 -> Row2
- SW19 pad 1: /Row3 -> Row3
- SW2 pad 1: /Row1 -> Row1
- SW20 pad 1: /Row4 -> Row4
- SW21 pad 1: /Row0 -> Row0
- SW22 pad 1: /Row1 -> Row1
- SW23 pad 1: /Row2 -> Row2
- SW24 pad 1: /Row3 -> Row3
- SW25 pad 1: /Row0 -> Row0
- SW26 pad 1: /Row1 -> Row1
- SW27 pad 1: /Row2 -> Row2
- SW28 pad 1: /Row3 -> Row3
- SW29 pad 1: /Row0 -> Row0
- SW3 pad 1: /Row2 -> Row2
- SW30 pad 1: /Row1 -> Row1
- SW31 pad 1: /Row2 -> Row2
- SW32 pad 1: /Row3 -> Row3
- SW33 pad 1: /Row0 -> Row0
- SW34 pad 1: /Row1 -> Row1
- SW35 pad 1: /Row2 -> Row2
- SW36 pad 1: /Row3 -> Row3
- SW37 pad 1: /Row0 -> Row0
- SW38 pad 1: /Row1 -> Row1
- SW39 pad 1: /Row2 -> Row2
- SW4 pad 1: /Row3 -> Row3
- SW40 pad 1: /Row3 -> Row3
- SW41 pad 1: /Row4 -> Row4
- SW42 pad 1: /Row0 -> Row0
- SW43 pad 1: /Row1 -> Row1
- SW44 pad 1: /Row2 -> Row2
- SW45 pad 1: /Row3 -> Row3
- SW46 pad 1: /Row4 -> Row4
- SW47 pad 1: /Row0 -> Row0
- SW48 pad 1: /Row1 -> Row1
- SW49 pad 1: /Row2 -> Row2
- SW5 pad 1: /Row4 -> Row4
- SW50 pad 1: /Row3 -> Row3
- SW51 pad 1: /Row4 -> Row4
- SW52 pad 1: /Row0 -> Row0
- SW53 pad 1: /Row1 -> Row1
- SW54 pad 1: /Row2 -> Row2
- SW55 pad 1: /Row3 -> Row3
- SW56 pad 1: /Row4 -> Row4
- SW6 pad 1: /Row0 -> Row0
- SW7 pad 1: /Row1 -> Row1
- SW8 pad 1: /Row2 -> Row2
- SW9 pad 1: /Row3 -> Row3
- U1 pad 1: /Row0 -> Net-(R4-Pad2)
- U1 pad 2: /Row1 -> GND
- U1 pad 5: /Col6 -> +5V
- U1 pad 6: /Col7 -> Net-(J1-PadA6)
Routing:
- net /Row0: track 432.4 -> 0.00 mm, vias 1 -> 0
- net /Row3: track 405.7 -> 0.00 mm, vias 2 -> 0
- net /Row1: track 404.2 -> 0.00 mm, vias 1 -> 0
- net Row3: track 0.00 -> 370.6 mm, vias 0 -> 1
- net Row2: track 0.00 -> 358.3 mm, vias 0 -> 1
- net /Row2: track 352.5 -> 0.00 mm
- net Row0: track 0.00 -> 342.2 mm, vias 0 -> 1
- net Row1: track 0.00 -> 336.6 mm, vias 0 -> 1
- net Row4: track 0.00 -> 291.6 mm, vias 0 -> 1
- net Col11: track 0.00 -> 275.8 mm, vias 0 -> 1
- net Col9: track 0.00 -> 274.0 mm, vias 0 -> 2
- net Col8: track 0.00 -> 265.1 mm
- net Col10: track 0.00 -> 260.9 mm, vias 0 -> 1
- net Col0: track 0.00 -> 254.0 mm, vias 0 -> 1
- net Col2: track 0.00 -> 244.2 mm, vias 0 -> 2
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- added copper zone on B.Cu, net GND
- added copper zone on F.Cu, net GND
Other:
- outline, holes or cut-outs redrawn
- net class Power added: clearance 0.2, trace_width 0.4, via_dia 0.8, via_drill 0.4
