File: Pteron56v0/Pteron56v0.sch (KiCad schematic (older format))
At the start: 113 parts, among them SW1 SW_PUSH, SW10 SW_PUSH, SW11 SW_PUSH, SW12 SW_PUSH, SW13 SW_PUSH, SW14 SW_PUSH, SW15 SW_PUSH, SW16 SW_PUSH, SW17 SW_PUSH, SW18 SW_PUSH, SW19 SW_PUSH, SW2 SW_PUSH, SW20 SW_PUSH, SW21 SW_PUSH, SW22 SW_PUSH, SW23 SW_PUSH, SW24 SW_PUSH, SW25 SW_PUSH, SW26 SW_PUSH, SW27 SW_PUSH, SW28 SW_PUSH, SW29 SW_PUSH, SW3 SW_PUSH, SW30 SW_PUSH, SW31 SW_PUSH, SW32 SW_PUSH, SW33 SW_PUSH, SW34 SW_PUSH, SW35 SW_PUSH, SW36 SW_PUSH, SW37 SW_PUSH, SW38 SW_PUSH, SW39 SW_PUSH, SW4 SW_PUSH, SW40 SW_PUSH, SW41 SW_PUSH, SW42 SW_PUSH, SW43 SW_PUSH, SW44 SW_PUSH, SW45 SW_PUSH, SW46 SW_PUSH, SW47 SW_PUSH, SW48 SW_PUSH, SW49 SW_PUSH, SW5 SW_PUSH, SW50 SW_PUSH, SW51 SW_PUSH, SW52 SW_PUSH, SW53 SW_PUSH, SW54 SW_PUSH, SW55 SW_PUSH, SW56 SW_PUSH, SW6 SW_PUSH, SW7 SW_PUSH, SW8 SW_PUSH, SW9 SW_PUSH, U1 ProMicro

Commit message: Add files via upload
Updates, added usb C 32u4-au
Parts:
- removed U1: ProMicro, Keyboard parts:Pro_Micro, symbol promicro:ProMicro
- added C?: 1u, Keyboard parts:.1uf_0805, symbol Device:C_Small
- added C? (x2): 22p, Keyboard parts:22pf_0603, symbol Device:C_Small
- added C? (x3): .1u, Keyboard parts:.1uf_0805, symbol Device:C_Small
- added C?: 10u, Keyboard parts:.1uf_0805, symbol Device:C_Small
- added D? (x56): LED, symbol Device:LED
- added F?: 500mA, symbol Device:Polyfuse_Small
- added J?: USB_C_Receptacle_USB2.0, Keyboard parts:USB-C-12-Pin-MidMount, symbol Connector:USB_C_Receptacle_USB2.0
- added Q?: 2N2219, Package_TO_SOT_THT:TO-39-3, symbol Transistor_BJT:2N2219
- added R: 10k, symbol Device:R
- added R? (x56): 1k, symbol Device:R
- added R? (x2): 22, Keyboard parts:1K_Resistor, symbol Device:R
- added R? (x2): 10k, Keyboard parts:10K_Resistor, symbol Device:R
- added R? (x2): 5.1k, Resistor_SMD:R_0603_1608Metric, symbol Device:R_Small
- added SW?: SW_PUSH, Keyboard parts:SW_SPST_TL3342, symbol keyboard_parts:SW_PUSH
- added U?: ATmega32U4-AU, Package_QFP:TQFP-44_10x10mm_P0.8mm, symbol MCU_Microchip_ATmega:ATmega32U4-AU
- added U?: USBLC6-2SC6, Package_TO_SOT_SMD:SOT-23-6, symbol Hruska:USBLC6-2SC6
- added X?: XTAL_GND, Keyboard parts:crystal_FA238-TSX3225, symbol keyboard_parts:XTAL_GND
Connections:
- net Col0: now also U?.10 (PB2)
- net Col1: now also U?.30 (PB6)
- net Col10: now also U?.28 (PB4)
- net Col2: now also U?.11 (PB3)
- net Col3: now also U?.9 (PB1)
- net Col4: now also U?.37 (PF6)
- net Col5: now also U?.36 (PF7)
- net Col6: now also U?.19 (PD1)
- net Col7: now also U?.18 (PD0)
- net Col8: now also U?.32 (PC7)
- net Col9: now also U?.27 (PD7)
- net Row0: now also U?.21 (PD3)
- net Row1: now also U?.20 (PD2)
- net Row2: now also U?.39 (PF4)
- net Row3: now also U?.25 (PD4)
- net Row4: now also U?.38 (PF5)
- net Col11 renamed +5V
- net +5V: now also C?.1, C?.1, C?.1, C?.1, F?.1, Q?.3 (C), R.2, R?.2, U?.1 (PE6), U?.14 (VCC), U?.2 (UVCC), U?.24 (AVCC), U?.34 (VCC), U?.44 (AVCC), U?.5 (VBUS), U?.7 (VBUS)
- new net: D?.1 (K), D?.1 (K), D?.1 (K), D?.1 (K), D?.1 (K), D?.1 (K), D?.1 (K), D?.1 (K), D?.1 (K), D?.1 (K), D?.1 (K), D?.1 (K), D?.1 (K), D?.1 (K), D?.1 (K), D?.1 (K), D?.1 (K), D?.1 (K), D?.1 (K), D?.1 (K), D?.1 (K), D?.1 (K), D?.1 (K), D?.1 (K), D?.1 (K), D?.1 (K), D?.1 (K), D?.1 (K), D?.1 (K), D?.1 (K), D?.1 (K), D?.1 (K), D?.1 (K), D?.1 (K), D?.1 (K), D?.1 (K), D?.1 (K), D?.1 (K), D?.1 (K), D?.1 (K), D?.1 (K), D?.1 (K), D?.1 (K), D?.1 (K), D?.1 (K), D?.1 (K), D?.1 (K), D?.1 (K), D?.1 (K), D?.1 (K), D?.1 (K), D?.1 (K), D?.1 (K), D?.1 (K), D?.1 (K), D?.1 (K), Q?.1 (E)
- new net: D?.2 (A), R?.1 (x55)
- new net: R?.2, R?.2, R?.2, R?.2, R?.2, R?.2, R?.2, R?.2, R?.2, R?.2, R?.2, R?.2, R?.2, R?.2, R?.2, R?.2, R?.2, R?.2, R?.2, R?.2, R?.2, R?.2, R?.2, R?.2, R?.2, R?.2, R?.2, R?.2, R?.2, R?.2, R?.2, R?.2, R?.2, R?.2, R?.2, R?.2, R?.2, R?.2, R?.2, R?.2, R?.2, R?.2, R?.2, R?.2, R?.2, R?.2, R?.2, R?.2, R?.2, R?.2, R?.2, R?.2, R?.2, R?.2, R?.2, R?.2
- new net: F?.2, J?.A4 (VBUS), J?.A9 (VBUS), J?.B4 (VBUS), J?.B9 (VBUS)
- new net: J?.A5 (CC1), R?.2
- new net: J?.A6 (D+), J?.B6 (D+), U?.6 (OUT1)
- new net: J?.A7 (D-), J?.B7 (D-), U?.4 (OUT2)
- new net: J?.B5 (CC2), R?.2
- new net: C?.1, U?.6 (UCAP)
- new net: R?.1, U?.3 (D-)
- new net: R?.2, U?.3 (IN2)
- new net: R?.1, U?.4 (D+)
- new net: R?.2, U?.1 (IN1)
- new net: R?.1, SW?.2, U?.13 (~RESET)
- new net: C?.1, U?.16 (XTAL2), X?.2
- new net: C?.1, U?.17 (XTAL1), X?.1
- new net: Q?.2 (B), R.1, U?.29 (PB5)
- new net: R?.2, U?.33 (~HWB~/PE2)
- new net GND: C?.2, C?.2, C?.2, C?.2, C?.2, C?.2, C?.2, J?.A1 (GND), J?.A12 (GND), J?.B1 (GND), J?.B12 (GND), J?.S1 (SHIELD), R?.1, R?.1, R?.1, SW?.1, U?.15 (GND), U?.2 (GND), U?.23 (GND), U?.35 (GND), U?.43 (GND), U?.5 (UGND), X?.3
- new net RX_LED: U?.8 (PB0)
- new net TX_LED: U?.22 (PD5)
- no-connect marks 0 -> 2
Other:
- moved on the sheet: D1, D10, D11, D12, D13, D14, D15, D16, D17, D18, D19, D2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

Commit message: Add files via upload
More edits, finished the MCU. 

TODO:
THT LEDs
WS2812b underglow
Add EC11 encoder
Parts:
- removed F?: 500mA, symbol Device:Polyfuse_Small
- removed J?: USB_C_Receptacle_USB2.0, Keyboard parts:USB-C-12-Pin-MidMount, symbol Connector:USB_C_Receptacle_USB2.0
- removed R? (x2): 5.1k, Resistor_SMD:R_0603_1608Metric, symbol Device:R_Small
- removed U?: USBLC6-2SC6, Package_TO_SOT_SMD:SOT-23-6, symbol Hruska:USBLC6-2SC6
- added F1: 500mA, Fuse:Fuse_0402_1005Metric, symbol Device:Polyfuse_Small
- added J1: USB_C_Receptacle_USB2.0, Connector_USB:USB_C_Receptacle_XKB_U262-16XN-4BVC11, symbol Connector:USB_C_Receptacle_USB2.0
- added R1, R2: 5.1k, Resistor_SMD:R_0603_1608Metric, symbol Device:R_Small
- added U1: USBLC6-2SC6, Package_TO_SOT_SMD:SOT-23-6, symbol Hruska:USBLC6-2SC6
- D100, D101, D102, D103, D104, D105, D106, D107, D108, D109, D110, D111, D112, D57, D58, D59, D60, D61, D62, D63, D64, D65, D66, D67, D68, D69, D70, D71, D72, D73, D74, D75, D76, D77, D78, D79, D80, D81, D82, D83, D84, D85, D86, D87, D88, D89, D90, D91, D92, D93, D94, D95, D96, D97, D98, D99: renamed from D?; footprint (none) -> LED_SMD:LED_0402_1005Metric
- R10, R11, R12, R13, R14, R15, R16, R17, R18, R19, R20, R21, R22, R23, R24, R25, R26, R27, R28, R29, R30, R31, R32, R33, R34, R35, R36, R37, R38, R39, R40, R41, R42, R43, R44, R45, R46, R47, R48, R49, R50, R51, R52, R53, R54, R55, R56, R57, R58, R59, R60, R61, R62, R63, R8, R9: renamed from R?; footprint (none) -> Resistor_SMD:R_0805_2012Metric
- R4, R5: renamed from R?; footprint Keyboard parts:1K_Resistor -> Keyboard parts:R_0805
- R7: renamed from R; footprint (none) -> Resistor_SMD:R_0805_2012Metric
- gave numbers to parts that had none: 13
Connections:
- net +5V: now also F1.1, U1.5 (VBUS); no longer D52.1 (K), D53.1 (K), D54.1 (K), D55.1 (K), D56.1 (K), U2.1 (PE6)
- net Col0: now also U2.32 (PC7); no longer U2.10 (PB2)
- net Col1: now also U2.31 (PC6); no longer U2.30 (PB6)
- net Col10: now also U2.30 (PB6); no longer U2.28 (PB4)
- net Col2: now also U2.38 (PF5); no longer U2.11 (PB3)
- net Col3: now also U2.39 (PF4); no longer U2.9 (PB1)
- net Col4: now also U2.40 (PF1); no longer U2.37 (PF6)
- net Col5: now also U2.41 (PF0); no longer U2.36 (PF7)
- net Col6: now also U2.11 (PB3); no longer U2.19 (PD1)
- net Col7: now also U2.25 (PD4); no longer U2.18 (PD0)
- net Col8: now also U2.26 (PD6); no longer U2.32 (PC7)
- net GND: now also J1.A1 (GND), J1.A12 (GND), J1.B1 (GND), J1.B12 (GND), J1.S1 (SHIELD), R1.1, R2.1, U1.2 (GND)
- net Row0: now also U2.10 (PB2); no longer U2.21 (PD3)
- net Row1: now also U2.9 (PB1); no longer U2.20 (PD2)
- net Row2: now also U2.20 (PD2); no longer U2.39 (PF4)
- net Row3: now also U2.21 (PD3); no longer U2.25 (PD4)
- net Row4: now also U2.37 (PF6); no longer U2.38 (PF5)
- net VCC: now also R10.2, R11.2, R12.2, R13.2, R14.2, R15.2, R16.2, R17.2, R18.2, R19.2, R20.2, R21.2, R22.2, R23.2, R24.2, R25.2, R26.2, R27.2, R28.2, R29.2, R30.2, R31.2, R32.2, R33.2, R34.2, R35.2, R36.2, R37.2, R38.2, R39.2, R40.2, R41.2, R42.2, R43.2, R44.2, R45.2, R46.2, R47.2, R48.2, R49.2, R50.2, R51.2, R52.2, R53.2, R54.2, R55.2, R56.2, R57.2, R58.2, R59.2, R60.2, R61.2, R62.2, R63.2, R8.2, R9.2
- net at R5.2: now also U1.3 (IN2)
- net at R4.2: now also U1.1 (IN1)
- net RX_LED: no longer names the net of U2.8 (PB0)
- net TX_LED: no longer names the net of U2.22 (PD5)
- new net: F1.2, J1.A4 (VBUS), J1.A9 (VBUS), J1.B4 (VBUS), J1.B9 (VBUS)
- new net: J1.A5 (CC1), R1.2
- new net: J1.A6 (D+), J1.B6 (D+), U1.6 (OUT1)
- new net: J1.A7 (D-), J1.B7 (D-), U1.4 (OUT2)
- new net: J1.B5 (CC2), R2.2
- new net Col11: D52.1 (K), D53.1 (K), D54.1 (K), D55.1 (K), D56.1 (K), U2.28 (PB4)
- no-connect marks 2 -> 3
